File: hardware_gnssbike/cad/folha1-energia.kicad_sch (KiCad schematic)
At the start: 55 parts, among them J101 Molex 2036150003, J102 JST SM06B-GHS-TB, U101 nPM1300-QEAA, U102 MAX17262REWL, U103 AEM10900, U104 TPS7A0218PDQN

Commit message: fix(hardware): fail the schematic check when a pin sits in two nets
A pin in two nets is a short, and the check merged the two nets instead of
complaining: U103's SDA was in both PWR_SDA and the 3V0 rail, which tied the
whole power bus to 3.0 V and shorted out R107, and the merge hid it. Now any
pin in two nets fails, except for the connectors declared in PASSA_DIRETO,
where a connector and the part behind it really are one node drawn as two.

Three more things the check then caught, all in the energy sheet:

  - the AEM10900's inductor had one end on a net of its own going nowhere.
    It boosts 1.67 V to 3.9 V, so the far end belongs on SRC; the open item
    now says to confirm it against figure 3 of DS-AEM10900-v1.6.0.
  - the flash's 22 uF bulk sat before the current jumper instead of beside
    the part, which is what 02-calculos.md asks for and what every other
    block on this board does.
  - four decoupling capacitors had no ground.

The unconnected pins are now written out one by one with the reason, so a
loose end is a decision on the page and not an absence.
Connections:
- net 3V0: no longer R107.2, U101.13 (SDA), U102.C1 (SDA), U103.13 (SDA)
- net GND: now also C107.2, C108.2, C109.2, C113.2
- net at C115.1, PV101.1 (P), PV102.1 (P)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: now also L103.1
- net at U103.5 (SW_DCDC): now also L103.2; no longer L103.1
- net at U103.8 (STO): no longer L103.2
- new net PWR_SDA: R107.2, U101.13 (SDA), U102.C1 (SDA), U103.13 (SDA)

Commit message: fix(hardware): the solar panel and the antenna had nowhere to touch the board
This board could not be built. The six solar modules live in the case and
connect to SRC and GND; the GNSS antenna element lives in the case wall and
connects to RF_ANT and GND. On the board, SRC reached only the harvester, its
capacitor and its inductor, and RF_ANT reached only the pi network. There was
no pad for either of them. The wires had nowhere to land.

04-pcb-e-caixa.md had already decided how they arrive - the antenna "com
contatos de mola" on line 271, the panels "em 3 grupos, mola ou FPC" on line
388 - and line 661 listed as open that "a area dos pads de mola e dos
conectores dos tres grupos de paineis nao esta dimensionada em lugar nenhum".
It is dimensioned now: two 2.0 x 2.0 mm gold pads at 3.0 mm pitch, with no
paste, because a spring presses on them and nothing is soldered.

J302 takes the antenna, just below its keep-out and a few millimetres from
the pi network, which is what the same document asks for when it says the
50 ohm line is "poucos mm". J103, J104 and J105 take the three groups of
panels, in the free bands of the two edges - computed, not guessed: the left
edge is taken by the light sensor, the two flat cables, the M2 hole, the
battery connector and a key. All three sit within about 15 mm of the
harvester, because SRC comes off a solar cell at high impedance and a long
run of it picks up everything.

The bodies stopped being identical black cuboids. What distinguishes these
packages at a glance is where the metal is, so a QFN now shows its exposed
pad and the ring of lead flags underneath, a SOIC stands on gull-wing leads
that reach out on two sides, a SOT has its three, and a wafer-level package
is bare silicon over a grid of balls. Each one carries the pin 1 dot. Every
dimension comes from the outline the footprint already had; what is new is
only which part of it is drawn as metal.

116 parts, no DRC error, 131 connections routed, and twelve of the thirteen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
Parts:
- added J103: contato de mola, 2 vias, gnssbike:ContatoMola_2x2mm_P3mm, symbol gnssbike:J103
- added J104: contato de mola, 2 vias, gnssbike:ContatoMola_2x2mm_P3mm, symbol gnssbike:J104
- added J105: contato de mola, 2 vias, gnssbike:ContatoMola_2x2mm_P3mm, symbol gnssbike:J105
Connections:
- net GND: now also J103.2 (N), J104.2 (N), J105.2 (N)
- net at C115.1, L103.1, PV101.1 (P)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: now also J103.1 (P), J104.1 (P), J105.1 (P)
Other:
- note added: "1 Energia - 58 posicoes. NADA MONTADO NEM MEDIDO."
- note removed: "1 Energia - 55 posicoes. NADA MONTADO NEM MEDIDO."
- moved on the sheet: C101, C102, C103, C104, C105, C106, C107, C108, C109, C110, C111, C112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

Commit message: feat(hardware): the test points, a readable silkscreen, and paper that fits
Eleven of the sixteen test points of 06-conectores-e-pontos-de-teste.md were
not on the board. Only the three of the console sheet existed; a rail you
cannot put a probe on is a rail you cannot debug. VBUS, VBUSOUT, VBAT, VSYS,
3V0, 1V8, SD3V0, 3V3BL, VBCKP, VINT and the ground reference are there now,
each beside the thing it measures, and each takes what is LEFT: placed with
the rest of JUNTO they pushed three decoupling capacitors off their rings,
one of them to 4.0 mm from a pin that wants 2. The two that are still
missing are the document's own absences - TP111 measures ST_STO, which the
AEM10900 datasheet does not have, and TP401 measures 5V0, from a regulator
not fitted with the JDI panel. The list lives in parts.TESTE and nets.py
refuses a point that names a net that does not exist.

The silkscreen named nothing. Every reference sat 1.8 mm above its part at
0.7 mm with a 0.1 mm stroke - below the floor every fab publishes - and 37
pairs of designators printed on top of each other. The text is at the fab
minimum now, 0.8 mm with 0.15, and each label is PLACED: candidates around
its own courtyard, nearest first, never over another label and preferably
not over another part's outline. 127 references, 0 overlapping. The mounting
hole's REF** is hidden; it names nothing and was the last label sitting on
another.

Ground: a mesh, not just a hem. Edge stitching keeps the boundary of the
surface pours from becoming a radiating slot and does nothing for the
middle, where a patch of pour that reaches the inner plane through a via
20 mm away is not ground at 2.4 GHz. A 4.0 mm grid of ground vias now
covers the board - under the 6.1 mm that is a tenth of a wavelength in
FR-4 - laid last, on what is free, so a stitch never costs a connection.

The router's search learned about pad fields. The neck beside a pad existed
only in emitir(), and emitir only ever sees paths the search already found,
so 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
Parts:
- added TP101: pad, TestPoint:TestPoint_Pad_D1.0mm, symbol gnssbike:TP101
- added TP102: pad, TestPoint:TestPoint_Pad_D1.0mm, symbol gnssbike:TP102
- added TP103: pad, TestPoint:TestPoint_Pad_D1.0mm, symbol gnssbike:TP103
- added TP104: pad, TestPoint:TestPoint_Pad_D1.0mm, symbol gnssbike:TP104
- added TP105: pad, TestPoint:TestPoint_Pad_D1.0mm, symbol gnssbike:TP105
- added TP106: pad, TestPoint:TestPoint_Pad_D1.0mm, symbol gnssbike:TP106
- added TP107: pad, TestPoint:TestPoint_Pad_D1.0mm, symbol gnssbike:TP107
- added TP108: pad, TestPoint:TestPoint_Pad_D1.0mm, symbol gnssbike:TP108
- added TP109: pad, TestPoint:TestPoint_Pad_D1.0mm, symbol gnssbike:TP109
- added TP110: pad, TestPoint:TestPoint_Pad_D1.0mm, symbol gnssbike:TP110
- added TP112: pad, TestPoint:TestPoint_Pad_D1.0mm, symbol gnssbike:TP112
Connections:
- net 1V8: now also TP106.1
- net 3V0: now also TP105.1
- net 3V3BL: now also TP108.1
- net GND: now also TP112.1
- net SD3V0: now also TP107.1
- net VBAT: now also TP103.1
- net VBCKP: now also TP109.1
- net VBUS: now also TP101.1
- net VBUSOUT: now also TP102.1
- net VINT: now also TP110.1
- net VSYS: now also TP104.1
Other:
- note added: "1 Energia - 69 posicoes. NADA MONTADO NEM MEDIDO."
- note removed: "1 Energia - 58 posicoes. NADA MONTADO NEM MEDIDO."
- moved on the sheet: C101, C102, C103, C104, C105, C106, C107, C108, C109, C110, C111, C112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

Commit message: feat(hardware): draw each part as its own symbol, not as a block
A rectangle with pin names down its sides is how an INTEGRATED CIRCUIT is
drawn, and only an integrated circuit. This generator drew all 127 parts
that way - resistors, ceramic capacitors, diodes, the TVS - and a sheet of
blocks joined by lines does not show a circuit.

Every class has its own symbol now, in the standard form, with the lead
axis on x and the body between -1.27 and +1.27 mm: a zigzag for a resistor
and a 0 ohm link (42 of them), two parallel plates for a ceramic capacitor
and a curved plate with a + for an electrolytic (31), four arcs for an
inductor (4), the same arcs inside a rectangle for a ferrite bead, which is
what tells the two apart, a zigzag with a diagonal arrow for the thermistor,
a triangle and a bar for a diode with arrows leaving it for an LED, two
contacts with a bar and a plunger for a key, a circle with a diagonal for
the buzzer, and a circle on the end of a lead for a test point. The 36 that
stay rectangles are the ones that should be: the ICs, the connectors and the
display. A two terminal part no longer prints pin numbers or pin names -
"1" and "2" on a resistor is noise, and the symbol already says which end is
which where it matters.

The power symbols had room reserved for the symbol and none for its NAME:
two ground pins two grid steps apart each got their own symbol, the symbols
did not collide, and the words printed over each other - "GNDGNDGND" along
the bottom of every chip. What is reserved now is the whole thing. With a
limit: the first cut let the stub run to fourteen grid steps looking for a
clear spot, and one of them crossed a component and split a net. A long stub
is worse than a crowded label, so it stops at eight and the label gives way.

One attempt is NOT in this commit, on purpose. Grouping every pin of a rail
on one edge into a single symbol - which is what a person draws - joins the
stubs with a line that runs along the part's edge and crosses w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
Other:
- moved on the sheet: D101, J103, J104, J105, U104

Commit message: feat(hardware): buy what JLCPCB can actually assemble
The board is made and assembled at JLCPCB, so every part has to be one
LCSC stocks - the owner's rule of 2026-09-24, with the Minew module and
the solar cells as the only exceptions. Three surveys against LCSC's
catalogue and JLCPCB's assembly API checked the 34 parts that are not a
plain resistor or capacitor, and this is what came back.

Parts that changed, and what each change costs:

  J101  Molex 2036150003 -> HRO TYPE-C-31-M-12 (C165948). 309 in the
        world at US$ 5,69 against 91.943 at US$ 0,186, and KiCad carries
        the land pattern under the part's own name. The body goes from
        8,58 to 7,35 mm, so the case opening changes.
  D101  ESD761DPYR -> TPD1E05U06DPYR (C436349). Same X1SON-2 and better
        capacitance, but bidirectional 24 V becomes unidirectional
        5,5 V: orientation now matters and a faulty cable putting 20 V
        on a CC line is no longer survivable.
  J103  three pairs of spring pads -> one JST ZH of 4 ways, with three
        0 ohm joining the groups to SRC. Nobody assembles a spring, a
        bicycle vibrates, and a pressed contact that opens and closes on
        the input of a switching converter is a dirty transient. ZH of
        1,5 mm on purpose: the cell is a GH of 1,25 and 4,2 V into the
        harvester's 2,73 V input would kill it. The 0 ohm let one face
        be measured alone in the sun.
  D105  new: a clamp on SRC. The right connector stops the mistake; the
        clamp stops the damage when the mistake comes from a crimp.
  J101  the shell had no pin, so four pads of the land pattern floated.

U101 and U103 stay as they are and go by consignment: the nPM1300 QFN is
zero on both sides and the whole e-peas line is zero. The nPM1300 does
exist in WLCSP-35, but its 0,419 x 0,440 mm ball pitch is smaller than
this board's 0,45 mm via and would force via-in-pad on every board ever
made, probably six layers, twice the thermal resistance and a light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
Parts:
- removed J104: contato de mola, 2 vias, gnssbike:ContatoMola_2x2mm_P3mm, symbol gnssbike:J104
- removed J105: contato de mola, 2 vias, gnssbike:ContatoMola_2x2mm_P3mm, symbol gnssbike:J105
- added D105: TVS 3,0 V, Diode_SMD:D_SOD-523, symbol gnssbike:D105
- added R113: 0 R, Resistor_SMD:R_0402_1005Metric, symbol gnssbike:R113
- added R114: 0 R, Resistor_SMD:R_0402_1005Metric, symbol gnssbike:R114
- added R115: 0 R, Resistor_SMD:R_0402_1005Metric, symbol gnssbike:R115
- D101: value ESD761DPYR -> TPD1E05U06DPYR
- J101: value Molex 2036150003 -> HRO TYPE-C-31-M-12; footprint Connector_USB:USB_C_Receptacle_Palconn_UTC16-G -> Connector_USB:USB_C_Receptacle_HRO_TYPE-C-31-M-12
- J103: value contato de mola, 2 vias -> JST S4B-ZR-SM4A-TF; footprint gnssbike:ContatoMola_2x2mm_P3mm -> Connector_JST:JST_ZH_S4B-ZR-SM4A-TF_1x04-1MP_P1.50mm_Horizontal
Connections:
- net GND: now also J101.S1 (SHELL), J103.4 (GND), D105.2 (GND); no longer J103.2 (N)
- new net: C115.1, D105.1 (IO), L103.1, R113.2, R114.2, R115.2, U103.28 (SRC)
- new net: J103.3 (PV_C), PV105.1 (P), PV106.1 (P), R115.1
- new net: J103.1 (PV_A), PV101.1 (P), PV102.1 (P), R113.1
- new net: J103.2 (PV_B), PV103.1 (P), PV104.1 (P), R114.1
Other:
- note added: "1 Energia - 71 posicoes. NADA MONTADO NEM MEDIDO."
- note removed: "1 Energia - 69 posicoes. NADA MONTADO NEM MEDIDO."
- moved on the sheet: C101, C102, C103, C104, C105, C106, C107, C108, C109, C110, C111, C112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

Commit message: feat(hardware): the solar harvester becomes the ADP5091
The whole e-peas line is zero at LCSC - 31 references, every one of them
- and this board is assembled at JLCPCB. DigiKey never sold the part
either, so consignment was a bet on a part nobody had confirmed is for
sale. The ADP5091ACPZ-2-R7 (C579259) does the same job and can be
bought.

It is not a drop-in. What it does keep: MPPT from 0,08 to 3,3 V, cold
start at 380 mV, a programmable charge threshold, and a programmable
discharge cut-off WITH a switch that really opens between the cell and
the system - which the AEM10900 did not have in that form.

What it loses, and both cost something:

  I2C. There is no bus at all: every threshold is a resistor divider.
  status.solar_mw leaves the screen or becomes an estimate from the net
  current the MAX17262 already measures, and the firmware's aem10900.c,
  361 lines, goes with its binding, its registers and its devicetree
  node.

  The NTC. The AEM10900 cut the charge outside 0 to 45 C by itself, in
  hardware. The ADP5091 has no temperature input at all, and this is
  now an OPEN DEFECT, not a solved problem. The obvious answer - a
  nanoamp comparator on the NTC driving DIS_SW - does not close: the
  divider would be permanently on, and 10 k against 22 k at 4,2 V is
  131 uA continuous, more than the whole device asleep. The four ways
  out are written down where the part is defined.

Three numbers decided the design:

  The inductor is 22 uH +-20 %, not a range - the internal peak control
  was dimensioned for it, and the data sheet says so twice. Isat must be
  30 % above the peak, so >= 390 mA with this variant. The 4,7 uH here
  was the AEM10900's and does not serve; the package grows from
  2,5 x 2,0 to 3 x 3 mm.

  The MPPT ratio is the BOTTOM resistor over the total, and inverting it
  puts the tracker at 0,19 instead of 0,81. 18 M below and 4,3 M above
  give 0,80717 against the 0,807 the panel wants: 0,9 mV of error, in
  E24 values, summing the same 2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
Parts:
- added C119: 10 nF, Resistor_SMD:R_0402_1005Metric, symbol gnssbike:C119
- added C120: 100 nF, Resistor_SMD:R_0402_1005Metric, symbol gnssbike:C120
- added C121: 4,7 uF, Resistor_SMD:R_0402_1005Metric, symbol gnssbike:C121
- added R116: 18 M, Resistor_SMD:R_0402_1005Metric, symbol gnssbike:R116
- added R117: 4,3 M, Resistor_SMD:R_0402_1005Metric, symbol gnssbike:R117
- added R118: 4,32 M, Resistor_SMD:R_0402_1005Metric, symbol gnssbike:R118
- added R119: 2,67 M, Resistor_SMD:R_0402_1005Metric, symbol gnssbike:R119
- added R120: 6,65 M, Resistor_SMD:R_0402_1005Metric, symbol gnssbike:R120
- added R121: 3,32 M, Resistor_SMD:R_0402_1005Metric, symbol gnssbike:R121
- added R122: 402 k, Resistor_SMD:R_0402_1005Metric, symbol gnssbike:R122
- added R123: 111 k, Resistor_SMD:R_0402_1005Metric, symbol gnssbike:R123
- L103: value 4,7 uH -> 22 uH
- U103: value AEM10900 -> ADP5091ACPZ-2
Connections:
- net 3V0: no longer U103.10 (I2C_VDD)
- net GND: now also U103.10 (AGND), U103.12 (PGND), U103.24 (REG_D0), U103.3 (SETBK), U103.EP (EPAD), C119.2, C120.2, C121.2, R116.2, R119.2, R121.2, R122.2, R123.2; no longer U103.1 (GND1), U103.17 (STO_CFG1), U103.29 (GND_PAD), U103.4 (GND2)
- net PWR_SCL: no longer U103.12 (SCL)
- net PWR_SDA: no longer U103.13 (SDA)
- net VBAT_SYS: now also U103.16 (SYS), U103.17 (BAT), C120.1, R118.1, R120.1
- net at C115.1, D105.1 (IO), L103.1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: now also TP110.1, U103.9 (VIN), R117.1; no longer U103.28 (SRC)
- net at R104.2, R105.1: now also U103.22 (DIS_SW); no longer U103.9 (DIS_STO_CH)
- net at R106.2, RT101.1: no longer U103.25 (TH_MON)
- net at R106.1: no longer U103.26 (TH_REF)
- net at L103.2: now also U103.13 (SW); no longer U103.5 (SW_DCDC)
- net at U103.11 (LLD): no longer R111.2
- net at U103.7 (MPPT): now also R116.1, R117.2
- net at U103.8 (CBP): now also C119.1
- removed net VINT: C116.1, TP110.1, U103.14 (KEEP_ALIVE), U103.15 (R_MPP1), U103.16 (T_MPP0), U103.18 (VINT2), U103.19 (STO_CFG0), U103.20 (R_MPP0), U103.21 (T_MPP1), U103.22 (STO_CFG2), U103.24 (R_MPP2), U103.6 (VINT)
- new net: R120.2, R121.1, U103.4 (SETSD)
- new net: C121.1, U103.14 (REG_OUT), U103.15 (REG_FB)
- new net: R123.1, U103.20 (VID)
- new net: R118.2, R119.1, U103.6 (TERM)
- new net: R122.1, U103.21 (MINOP)
Other:
- note added: "1 Energia - 82 posicoes. NADA MONTADO NEM MEDIDO."
- note removed: "1 Energia - 71 posicoes. NADA MONTADO NEM MEDIDO."
- moved on the sheet: C101, C102, C103, C104, C105, C106, C107, C108, C109, C110, C111, C112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

Commit message: feat(hardware): real symbols and real 3D models, from KiCad's own libraries
Two of the owner's asks in one commit, because they turned out to be the
same idea: stop drawing what already exists, reviewed, in the library.

THE SCHEMATIC. 36 of the parts were rectangles with pins around them - the
ICs, the connectors and the display - and a rectangle says nothing. Anyone
reading a schematic recognises a coaxial connector by the circle with the
dot, a switch by the contact that opens, a MOSFET by the channel and the
arrow.

ksym.py reads a symbol out of KiCad's own library - 21.110 of them, every
one reviewed against the KLC - and embeds it in our schematic with our
properties. simbolos.py says which part uses which. Eleven are in, and
ksym.checar() verifies every one pin number by pin number, because a
pretty symbol with the wire on the wrong pin is worse than a correct
rectangle. RF_GPS:MAX-M10S is literally our receiver: 18 pins, 18 names,
the same LCC-18.

Three symbols verify clean and still break the drawing, and they are
parked with the reason MEASURED rather than "did not work": the ADP5091
puts MPPT on the bottom edge beside its three ground pins and the ground
power symbol lands on the MPPT wire; the USB-C stacks four contacts per
point with 5,08 mm stubs and VBUS meets CC1; the ten pins of the display
FPC are all on one edge and two wires cannot reach. Each needs work
somewhere else - the power symbol placer, the placement - not a different
symbol.

Three bugs were found and fixed on the way, all in the router, all of the
same family: it assumed things about symbols that are only true of the
ones this project draws.

  - Symbols from KiCad are NOT centred on their origin. A
    Conn_01x10_Socket has its drawing at x -1,27 to 0 and all ten pins at
    x = -5,08. Treated as centred, pins fall inside the obstacle, the
    router cannot reach them from outside and goes over them instead -
    and two nets that touch are one net, with nothing in the drawing
    sa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
Parts:
- U103: footprint Package_DFN_QFN:QFN-28-1EP_4x4mm_P0.4mm_EP2.3x2.3mm -> Package_CSP:LFCSP-24-1EP_4x4mm_P0.5mm_EP2.3x2.3mm
Connections:
- net GND: now also U103.25 (EPAD); no longer U103.EP (EPAD)
Other:
- moved on the sheet: C101, C102, C103, C104, C105, C106, C107, C108, C109, C110, C111, C112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

Commit message: fix(hardware): the debug connector had RESET on the wrong contact
This one would have cost a board. The Tag-Connect TC2030 footprint had
pin 3 as no-connect and RESET on pin 6. The manufacturer's own data
sheet, TC2030-CTX_1.pdf, table "Connections", says the opposite: on the
six-pin footprint it is 3 = nRESET and 6 = SWO/TDO.

Where the mistake came from is worth writing down, because it is easy to
make twice: 1 VCC, 2 SWDIO, 3 GND, 4 SWCLK, 5 GND, 6 SWO is the
numbering of the ten-way Cortex header on the PROBE side, not of the
six-pin footprint on the board. Mixing the two gives exactly what was
written here.

What it would have done: the probe's nRESET is an open drain output, so
it would have driven nothing, and the MCU's reset would have hung off
the probe's SWO INPUT. Nothing burns - SWO runs target to probe, there
is no short - but the debugger can never reset the target: no connect
under reset, no pin reset. On an nRF54LM20A that reboots from task_wdt
or reconfigures its SWD pins, that removes the standard way out and
leaves only a full CTRL-AP erase.

The documentation carried a worse version still. 06 had GND on contact 3,
which fabricated would tie the probe's open-drain nRESET to copper
ground and hold the target in reset forever.

The project's own notes had predicted this exact variant - 06 carried a
CAUTION saying so and README an open checklist item. It was that one, and
it was caught before layout. Both are now closed, and the connector's
pin 6 is recorded as SWO with what is still unknown about it: which pad
of the ME54BS13 exposes SWO, which would give printf over ITM during
bring-up.

Fixed in parts.py, nets.py, 03-netlist.md, 06-conectores-e-pontos-de-teste.md,
07-sequencias-e-protecao.md and README.md.

Verified: check_sch and check_pcb pass, 78 of 78 diagrams render, 1529
links and none broken.
Other:
- moved on the sheet: C101, C102, C103, C104, C105, C106, C107, C108, C109, C110, C111, C112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
