File: hardware_gnssbike/cad/folha1-energia.kicad_sch (KiCad schematic)
At the start: 82 parts, among them J101 HRO TYPE-C-31-M-12, J102 JST SM06B-GHS-TB, J103 JST S4B-ZR-SM4A-TF, U101 nPM1300-QEAA, U102 MAX17262REWL, U103 ADP5091ACPZ-2, U104 TPS7A0218PDQN

Commit message: fix(hardware): six pins of the solar harvester were swapped
The second board-killing mistake of the day, and it was caught the same
way as the first: two sources disagreed, and the data sheet decided.

A first reading of the ADP5091 data sheet swapped SIX pins, in two
permutations of three - 2/4/6 (SETHYST, SETSD, TERM) and 7/9/10 (MPPT,
VIN, AGND). It only surfaced because KiCad's own Battery_Management:
ADP5091 symbol disagreed, and because the symbol check had just been
taught to compare pin NAMES and not only numbers. The numbers matched;
the signals did not.

Table 5, pages 8 and 9 of Rev. A (D14145-0-5/17(A)), with Figure 3
confirming side by side, says KiCad is right on all 24. Three
independent readings closed it: the table rebuilt from the geometry of
its columns, the self-consistency of each description - the one for pin
2 says "the SETSD pin", the one for pin 6 says "between SETPG and
SETHYST" - and Figure 3.

What would have gone to copper: the MPPT divider on pin 7, which is
AGND, shorted to analogue ground; the harvester with its 22 uH inductor
and 10 uF capacitor on pin 9, which is MPPT; and ground on pin 10, which
is the input.

The exposed pad is recorded as the data sheet has it: no number at all -
its row in Table 5 has the column empty - and "must be connected to
AGND". The 25 is a CAD convention, which is how KiCad's footprint
numbers it and how its symbol names it, stacked on pin 7.

Beware the preliminary Rev. PrA: its Table 5 swaps 14 and 17 and
contradicts its own Figure 2. It is good for nothing.

With the pinout right, the ADP5091 symbol goes in: 15 KiCad symbols now,
all verified pin number AND pin name.

Verified: check_sch and check_pcb pass, schematic and board agree.
Connections:
- net GND: now also U103.7 (AGND); no longer U103.10 (AGND)
- net at C115.1, D105.1 (IO), L103.1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: now also U103.10 (VIN); no longer U103.9 (VIN)
- net at R120.2, R121.1: now also U103.2 (SETSD); no longer U103.4 (SETSD)
- net at R116.1, R117.2: now also U103.9 (MPPT); no longer U103.7 (MPPT)
- net at R118.2, R119.1: now also U103.4 (TERM); no longer U103.6 (TERM)
Other:
- moved on the sheet: C101, C102, C103, C104, C105, C106, C107, C108, C109, C110, C111, C112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

Commit message: feat(hardware): the ERC runs, and 52 hidden errors became 4 deliberate ones
check_sch.py compared our netlist against the one KiCad extracts, pin by
pin, and was good at that and blind to everything else. KiCad's own ERC
had never been run on this schematic. It found 52 errors, and among them
a capacitor with BOTH terminals in the air.

They were of four kinds, and three of them were the drawing failing to
say what it meant rather than the circuit being wrong:

  34 open pins with no flag. The NC pins of the ESD array, the GPIOs
  nobody uses, the receiver's SDA and SCL - it speaks UART - the
  programmer's SWO. Every one of them deliberate, and indistinguishable
  from a forgotten wire. They now carry a no-connect flag, taken from
  nets.py, which is already the source of truth about what is open: a
  pin that appears in no net is open, full stop. A net with a single pin
  counts as open too, which is what R111 became when the harvester
  changed and its pull-up lost its job.

  12 rails with no source the ERC could see. The 1V8_GNSS comes from
  1V8 through a ferrite, the SD3V0_FLASH from SD3V0 through a jumper,
  the harvester's VIN from the panel. PWR_FLAG is the symbol that exists
  to say "this is supplied, I answer for it". One per ELECTRICAL GROUP,
  not per net and not per sheet: two nets that share a pin are one net
  to KiCad - the display connector carries FPC_VSS on one side and GND
  on the other through the same contact - and a flag on each side would
  be two supply outputs wired together, which is another error.

  The last one needed the electrical type to come from the symbol that
  actually reaches the sheet. The four VBUS contacts of the USB-C are
  power_out in our parts.py and passive in KiCad's symbol, so the rule
  believed the rail had a source when it had none.

What is left is four violations, and all four are the same thing: two
supply OUTPUTS wired together. KiCad calls that an error by default
because in signal circuitry two outputs on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
Connections:
- no-connect marks 0 -> 26

Commit message: feat(hardware): GNSS receiver on the 3V0 rail, and the electrical items closed with the owner
The receiver ran at 1.8 V from BUCK1 through a TXU0204 level shifter, and
table 35 of the MAX-F10S integration manual asks +-2 % of a 1.8 V supply
where the nPM1300 buck gives +-5 %. A +-1 % LDO from 3V0 fixed the
tolerance and cost 35 mW at the battery (the receiver paid at 3.0 V with
1.2 V burnt in the LDO); option 1 of the same table - VCC and V_IO tied at
3.0 V, VIO_SEL open - costs 11 mW and removes the shifter. The owner chose
option 1. The receiver now sits on 3V0 through JP103 and the ferrite, the
four digital lines go pin to pin, the shifter and the LDO leave with four
capacitors, and BUCK1 stays fitted and unloaded as in configuration 1 of
the nPM1300 datasheet (the datasheet only shows an unused BUCK2, and what
it does not show is not copied). The devicetree follows: vcc-supply on
BUCK2, BUCK1 regulator-boot-off. The receiver no longer has a rail that
switches off; that consequence is recorded in docs/10.

Closed the same day, each a decision of the owner or a datasheet fact:

  - the ADP5091 TERM and SETSD dividers hung from BAT with REF open;
    figure 42 of the datasheet hangs all four external dividers from REF,
    which the chip switches to BAT with the hysteresis resistor in series.
    Equation 6 did not hold as drawn. Net ADP_REF, same values.
  - the solar charge thermal cut-off: the ADP5091 has no temperature
    input and the NTC divider was on the board with nobody reading it. A
    TLV7031 fed from the panel compares RT101/R106 with half of SRC and
    pulls DIS_SW high through a BAT54WS, in diode-OR with the USB divider.
    Hot side only; charging below 0 C stays open, and says so.
  - the centre key reaches P1.27 through a Schottky (D107): the SHPHLD
    node rises to 5.5 V with the cable.
  - J102 copper matched to the pinout 06 sends to the pack maker: the
    copper had VBAT+ on 1, NTC on 4, GND on 6 and 2, 3 and 5 open.
  - FB301 with 150 mO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
Parts:
- removed C112: 2,2 uF, Capacitor_SMD:C_0603_1608Metric, symbol gnssbike:C112
- removed R111: 10 k, Resistor_SMD:R_0402_1005Metric, symbol gnssbike:R111
- added C122: 100 nF, Capacitor_SMD:C_0603_1608Metric, symbol gnssbike:C122
- added C123: 100 nF, Capacitor_SMD:C_0603_1608Metric, symbol gnssbike:C123
- added C124: 100 nF, Capacitor_SMD:C_0603_1608Metric, symbol gnssbike:C124
- added C125: 100 nF, Capacitor_SMD:C_0603_1608Metric, symbol gnssbike:C125
- added C126: 100 nF, Capacitor_SMD:C_0603_1608Metric, symbol gnssbike:C126
- added C129: 100 nF, Capacitor_SMD:C_0603_1608Metric, symbol gnssbike:C129
- added D106: BAT54WS-7-F, Diode_SMD:D_SOD-323, symbol gnssbike:D106
- added D107: BAT54WS-7-F, Diode_SMD:D_SOD-323, symbol gnssbike:D107
- added R124: 100 k, Resistor_SMD:R_0402_1005Metric, symbol gnssbike:R124
- added R125: 100 k, Resistor_SMD:R_0402_1005Metric, symbol gnssbike:R125
- added U105: TLV7031DCKR, Package_TO_SOT_SMD:SOT-353_SC-70-5, symbol gnssbike:U105
- D105: value TVS 3,0 V -> PESD3V3S1UB-N
- R105: value 1 M -> 180 k
- R106: value 22 k -> 4,87 k
Connections:
- net 1V8: no longer JP103.1
- net 3V0: now also JP103.1, C129.1; no longer R112.1
- net 3V0_SENS: now also R112.1, C123.1, C124.1, C125.1, C126.1
- net GND: now also J102.2 (Pin_2), J102.5 (Pin_5), R106.2, C122.2, C123.2, C124.2, C125.2, C126.2, C129.2, R125.2, U105.2 (GND); no longer J102.6 (Pin_6), RT101.2
- net KEY_C_SW: now also D107.1 (K)
- net USB_DM: now also D102.6 (NC1)
- net USB_DP: now also D102.7 (NC2)
- net VBAT: now also C122.1
- net VBAT_CELULA: now also J102.6 (Pin_6)
- net VBAT_SYS: now also C116.1; no longer R118.1, R120.1
- net VSYS: now also U105.5 (V+)
- net at C115.1, D105.1 (IO), L103.1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: now also RT101.1, R124.1
- net at R104.2, R105.1, U103.22 (DIS_SW): now also D106.1 (K)
- net at U101.18 (NTC): now also J102.3 (Pin_3); no longer J102.4 (Pin_4)
- net at D102.1 (D1P), J101.A5 (CC1), U101.23 (CC1): now also D102.10 (NC4)
- net at D102.2 (D1N), J101.B5 (CC2), U101.24 (CC2): now also D102.9 (NC3)
- net at R106.1: now also RT101.2, U105.1 (IN+)
- net at U103.1 (REF): now also R118.1, R120.1
- net 1V8_BLOCO renamed 3V0_BLOCO
- new net: D106.2 (A), U105.4 (OUT)
- new net: R124.2, R125.1, U105.3 (IN-)
- new net KEY_C_D: D107.2 (A)
- no-connect marks 26 -> 14
Other:
- note added: "1 Energia - 91 posicoes. NADA MONTADO NEM MEDIDO."
- note removed: "1 Energia - 82 posicoes. NADA MONTADO NEM MEDIDO."
- moved on the sheet: C101, C102, C103, C104, C105, C106, C107, C108, C109, C110, C111, C113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

Commit message: feat(hardware): draw the schematic by functional block, the way a person reads it
The owner asked for an industrial-standard schematic: wires and labels,
A4 or A3 pages, the right symbols and values, easy to read, the circuits
subdivided by dashed boxes. Until now each sheet was the netlist drawn as
wires - parts on a grid in connection order and a maze router pulling a
wire from every pin to wherever its other end was, across the page.

blocos.py turns each sheet into a row of functional blocks in the order
the signal flows, each in a dashed rectangle with a title: on the power
sheet, USB-C and protection, the nPM1300, the gauge and the cell, the GNSS
backup, the solar harvester, the thermal cut-off. Membership comes from
the BLOCOS table (the anchors), then make_pcb.DECOPLA and JUNTO (the
board already says whose each capacitor is), then sheets.SEGUE, then the
netlist without rails, nearest anchor by hops. Inside a block the anchor
sits in the middle and each passive beside the pin it serves, on the
side that pin faces, mirrored when the pin that serves the chip is the
far one; parts that touch only rails go to a shelf under the chip. Rails
are power symbols, neighbouring pins of one rail get a wire along their
tips and one symbol; a net that leaves its block is a local label, one
that leaves the sheet a hierarchical label, both on a short stub the
maze router bends when the straight way is taken. Sheet 1 is A3, the
rest A4, measured by the drawing itself. Decoupling capacitors now live
on their chip's sheet whatever their number.

Three KiCad 8 facts were measured with kicad-cli's netlist export on the
way, because the first version assumed each one wrong and check_sch.py
caught it: (mirror x) swaps left for right, not (mirror y); a local label
named after a rail is the net /sheet/RAIL, another net; and a pin in the
middle of a long wire is not on it - "wires connect with other wires or
pins only if their ends coincide exactly" (Eeschema manual). The
conventions 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
Parts:
- removed C123: 100 nF, Capacitor_SMD:C_0603_1608Metric, symbol gnssbike:C123
- removed C124: 100 nF, Capacitor_SMD:C_0603_1608Metric, symbol gnssbike:C124
- removed C125: 100 nF, Capacitor_SMD:C_0603_1608Metric, symbol gnssbike:C125
- removed C126: 100 nF, Capacitor_SMD:C_0603_1608Metric, symbol gnssbike:C126
- removed D107: BAT54WS-7-F, Diode_SMD:D_SOD-323, symbol gnssbike:D107
- removed JP102: 0 R, Resistor_SMD:R_0402_1005Metric, symbol gnssbike:JP102
- removed JP103: 0 R, Resistor_SMD:R_0402_1005Metric, symbol gnssbike:JP103
- removed JP104: 0 R, Resistor_SMD:R_0402_1005Metric, symbol gnssbike:JP104
- removed JP105: 0 R, Resistor_SMD:R_0402_1005Metric, symbol gnssbike:JP105
- removed R107: 4,7 k, Resistor_SMD:R_0402_1005Metric, symbol gnssbike:R107
- removed R108: 4,7 k, Resistor_SMD:R_0402_1005Metric, symbol gnssbike:R108
- removed R112: 10 k, Resistor_SMD:R_0402_1005Metric, symbol gnssbike:R112
Connections:
- net 3V0 is gone; now on net 1V8: C105.1, C106.1, C107.1, C108.1, C129.1, L102.2, R109.1, R110.1, TP105.1, U101.12 (VDDIO), U101.28 (LSIN1), U101.32 (VOUT2)
- net 3V3BL is gone; now on net 1V8: C111.1, TP108.1, U101.31 (LSOUT2)
- net GND is gone; now on net 1V8: C101.2, C102.2, C103.2, C104.2, C105.2, C106.2, C107.2, C108.2, C109.2, C110.2, C111.2, C113.2, C114.2, C115.2, C116.2, C117.2, C118.2, C119.2, C120.2, C121.2, C122.2, C129.2, D101.2 (GND), D102.3 (GND1), D102.8 (GND2), D105.2 (GND), J101.A1 (GND), J101.A12 (GND), J101.B1 (GND), J101.B12 (GND), J101.S1 (SHIELD), J102.2 (Pin_2), J102.5 (Pin_5), J103.4 (Pin_4), PV101.2 (N), PV102.2 (N), PV103.2 (N), PV104.2 (N), PV105.2 (N), PV106.2 (N), R102.2, R103.2, R105.2, R106.2, R116.2, R119.2, R121.2, R122.2, R123.2, R125.2, TP112.1, U101.2 (PVSS1), U101.33 (AVSS), U101.6 (PVSS2), U102.C3 (GND), U103.12 (PGND), U103.23 (REG_D1), U103.24 (REG_D0), U103.25 (AGND), U103.3 (SETBK), U103.7 (AGND), U104.2 (GND), U104.5 (PAD), U105.2 (GND)
- net VBAT is gone; now on net SD3V0: C122.1, JP101.2, TP103.1, U102.A1 (TH), U102.A2 (BATT)
- net VBAT_SYS is gone; now on net 1V8: C102.1, C113.1, C116.1, C117.1, C120.1, U101.19 (VBAT), U102.B3 (SYS), U103.16 (SYS), U103.17 (BAT), U104.3 (EN), U104.4 (IN)
- net VBCKP is gone; now on net 1V8: C114.1, TP109.1, U104.1 (OUT)
- net VBUSOUT is gone; now on net 1V8: C110.1, R104.1, TP102.1, U101.22 (VBUSOUT)
- net VSYS is gone; now on net 1V8: C103.1, D103.2 (A), D104.2 (A), TP104.1, U101.20 (VSYS), U101.30 (LSIN2), U101.4 (PVDD), U105.5 (V+)
- net SRC: now reaches C115.1, D105.1 (IO), L103.1, R113.2, R114.2, R115.2, R117.1, R124.1, RT101.1, TP110.1, U103.10 (VIN)
- net DIS_SW: now reaches D106.1 (K), R104.2, R105.1, U103.22 (DIS_SW)
- net NTC_BAT: now reaches J102.3 (Pin_3), U101.18 (NTC)
- net CC1: now reaches D102.1 (D1P), D102.10 (NC4), J101.A5 (CC1), U101.23 (CC1)
- net CC2: now reaches D102.2 (D1N), D102.9 (NC3), J101.B5 (CC2), U101.24 (CC2)
Other:
- note added: "1 Energia - 79 posicoes. NADA MONTADO NEM MEDIDO."
- note added: "Backup do receptor GNSS"
- note added: "Colheita solar ADP5091"
- note added: "Corte termico da carga solar"
- note added: "Medidor de bateria e celula"
- note added: "USB-C e protecao"
- note added: "nPM1300: entrada, carga e os dois bucks"
- note removed: "1 Energia - 91 posicoes. NADA MONTADO NEM MEDIDO."
- moved on the sheet: C101, C102, C103, C104, C105, C106, C107, C108, C109, C110, C111, C113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
